File: pcb/fatbee_virtual_grid.kicad_pcb (KiCad board)
At the start: 2 copper layers, 302 x 112.5 mm, 168 parts, among them J1 Conn_01x07_Pin, J2 Conn_01x07_Pin, J3 Conn_01x03_Pin

Commit message: four thousand holes in Blackburn Lancashire
Parts:
- removed the REF** at (238.6, 61.8)
- removed the REF** at (313.5, 76.7)
- removed the REF** at (251.9, 99.7)
- removed the REF** at (65.7, 101.6)
- removed the REF** at (99.0, 124.4)
- removed the REF** at (293.2, 95.9)
- added REF**: M2, MountingHole:MountingHole_2.2mm_M2_DIN965, F.Cu at (154.0, 140.5)
- added REF**: M2, MountingHole:MountingHole_2.2mm_M2_DIN965, F.Cu at (226.0, 141.0)
- moved REF** 39.1 mm to (97.0, 115.5)
- moved REF** 28.8 mm to (67.5, 84.5)
- moved REF** 20.9 mm to (111.5, 79.0)
- moved REF** 17.5 mm to (140.5, 120.0)
- moved REF** 7.18 mm to (337.1, 79.0)
- moved REF** 4.27 mm to (40.6, 79.0)
